Commit message: Adapted URDF to be loaded into Gazebo

File: kr_robot_description/kr810/urdf/kr810_description.urdf.xacro (robot description, xacro)
@@ -86,5 +86,5 @@
         <origin xyz="0 0 0" rpy="0 0 0" />
         <geometry>
-          <mesh filename="package://kr_robot_description/kr810/meshes/a810/a810_Base.stl" scale="0.001 0.001 0.001"/>
+          <mesh filename="$(find kr_robot_description)/kr810/meshes/a810/a810_Base.stl" scale="0.001 0.001 0.001"/>
         </geometry>
         <material name="">
@@ -126,5 +126,5 @@
         <origin xyz="0 0 0.169" rpy="0 0 0" />
         <geometry>
-          <mesh filename="package://kr_robot_description/kr810/meshes/a810/a810_Link2.stl" scale="0.001 0.001 0.001"/>
+          <mesh filename="$(find kr_robot_description)/kr810/meshes/a810/a810_Link2.stl" scale="0.001 0.001 0.001"/>
         </geometry>
         <material name="">
@@ -164,5 +164,5 @@
         <origin xyz="0.049 0 0" rpy="-${pi/2} 0 -${pi/2}" />
         <geometry>
-          <mesh filename="package://kr_robot_description/kr810/meshes/a810/a810_Link3.stl" scale="0.001 0.001 0.001"/>
+          <mesh filename="$(find kr_robot_description)/kr810/meshes/a810/a810_Link3.stl" scale="0.001 0.001 0.001"/>
         </geometry>
         <material name="">
@@ -188,5 +188,5 @@
         <origin xyz="-0.05 -0.0 0.315" rpy="${pi/2} 0 -${pi/2}" />
         <geometry>
-          <mesh filename="package://kr_robot_description/kr810/meshes/a810/a810_Link4.stl" scale="0.001 0.001 0.001"/>
+          <mesh filename="$(find kr_robot_description)/kr810/meshes/a810/a810_Link4.stl" scale="0.001 0.001 0.001"/>
         </geometry>
         <material name="">
@@ -226,5 +226,5 @@
         <origin xyz="0.04 0.0005 0.0" rpy="-${pi/2} 0 ${pi/2}" />
         <geometry>
-          <mesh filename="package://kr_robot_description/kr810/meshes/a810/a810_Link5.stl" scale="0.001 0.001 0.001"/>
+          <mesh filename="$(find kr_robot_description)/kr810/meshes/a810/a810_Link5.stl" scale="0.001 0.001 0.001"/>
         </geometry>
         <material name="">
@@ -247,5 +247,5 @@
         <origin xyz="0.0 0.002 0.1035" rpy="0 0 -${pi/2}" />
         <geometry>
-          <mesh filename="package://kr_robot_description/kr810/meshes/a810/a810_Link6.stl" scale="0.001 0.001 0.001"/>
+          <mesh filename="$(find kr_robot_description)/kr810/meshes/a810/a810_Link6.stl" scale="0.001 0.001 0.001"/>
         </geometry>
         <material name="">
@@ -287,5 +287,5 @@
         <origin xyz="0.0 0.0 0.0" rpy="0 0 0" />
         <geometry>
-          <mesh filename="package://kr_robot_description/kr810/meshes/a810/a810_Link7.stl" scale="0.001 0.001 0.001"/>
+          <mesh filename="$(find kr_robot_description)/kr810/meshes/a810/a810_Link7.stl" scale="0.001 0.001 0.001"/>
         </geometry>
         <material name="">
@@ -303,5 +303,5 @@
         <origin xyz="0.0 -0.0 0.0" rpy="0 0 0" />
         <geometry>
-          <mesh filename="package://kr_robot_description/kr810/meshes/a810/a810_ToolIO.stl" scale="0.001 0.001 0.001"/>
+          <mesh filename="$(find kr_robot_description)/kr810/meshes/a810/a810_ToolIO.stl" scale="0.001 0.001 0.001"/>
         </geometry>
         <material name="">

Commit message: Got the gazebo sim control hardware plugin to function, at least

File: kr_robot_description/kr810/urdf/kr810_description.urdf.xacro (robot description, xacro)
@@ -421,192 +421,80 @@
     <child link="base"/>
   </joint>
-  <!-- Deprecated for Gazebo Harmonic -->
-  <!-- <gazebo>
-      <plugin filename="libgazebo_ros_control.so" name="ros_control">
-          <robotNamespace>/kr2_robot</robotNamespace>
-     </plugin>
-  </gazebo> -->
-  <!-- Following material setting relies on Ogre which is not supported anymore by Gazebo Harmonic -->
-  <!-- <gazebo reference="base">
-    <material>Gazebo/Black</material>
-  </gazebo>
-  <gazebo reference="link1">
-    <material>Gazebo/Grey</material>
-  </gazebo>
-  <gazebo reference="link2">
-    <material>Gazebo/White</material>
-  </gazebo>
-  <gazebo reference="link3">
-    <material>Gazebo/Grey</material>
-  </gazebo>
-  <gazebo reference="link4">
-    <material>Gazebo/White</material>
-  </gazebo>
-  <gazebo reference="link5">
-    <material>Gazebo/Grey</material>
-  </gazebo>
-  <gazebo reference="link6">
-    <material>Gazebo/White</material>
-  </gazebo>
-  <gazebo reference="end_effector">
-    <material>Gazebo/Black</material>
-  </gazebo> -->
-  <ros2_control name="kr810_system" type="gz_ros2_control::GazeboSimSystemInterface">
+  <ros2_control name="GazeboSimSystem" type="system">
     <hardware>
-      <plugin>gz_ros2_control/GazeboSimSystem</plugin> <!-- Changed from gazebo_ros2_control/GazeboSystem to gz_ros2_control/GazeboSimSystem -->
-      <!-- <plugin>kr_robot_driver/RobotSystem</plugin> Expected usage for real robot! -->
-      <param name="joints">
-        joint_1 joint_2 joint_3 joint_4 joint_5 joint_6 joint_7
-      </param>
-      <param name="command_interfaces">effort</param>
-      <param name="state_interfaces">position velocity</param>
-      <param name="use_sim_time">true</param>
+      <!-- Gazebo Harmonic backend -->
+      <plugin>gz_ros2_control/GazeboSimSystem</plugin>
     </hardware>
-    <!-- Each joint: effort-based control -->
+    <!-- 7 revolute joints, position command -->
     <joint name="joint_1">
-      <command_interface name="effort"/>
-      <state_interface name="position"/>
+      <command_interface name="position">
+      </command_interface>
+      <state_interface name="position">
+        <param name="initial_value">1.0</param>
+      </state_interface>
       <state_interface name="velocity"/>
     </joint>
     <joint name="joint_2">
-      <command_interface name="effort"/>
-      <state_interface name="position"/>
+      <command_interface name="position">
+      </command_interface>
+      <state_interface name="position">
+        <param name="initial_value">-1.0</param>
+      </state_interface>
       <state_interface name="velocity"/>
     </joint>
     <joint name="joint_3">
-      <command_interface name="effort"/>
-      <state_interface name="position"/>
+      <command_interface name="position">
+      </command_interface>
+      <state_interface name="position">
+        <param name="initial_value">1.0</param>
+      </state_interface>
       <state_interface name="velocity"/>
     </joint>
     <joint name="joint_4">
-      <command_interface name="effort"/>
-      <state_interface name="position"/>
+      <command_interface name="position">
+      </command_interface>
+      <state_interface name="position">
+        <param name="initial_value">1.0</param>
+      </state_interface>
       <state_interface name="velocity"/>
     </joint>
     <joint name="joint_5">
-      <command_interface name="effort"/>
-      <state_interface name="position"/>
+      <command_interface name="position">
+      </command_interface>
+      <state_interface name="position">
+        <param name="initial_value">1.0</param>
+      </state_interface>
       <state_interface name="velocity"/>
     </joint>
     <joint name="joint_6">
-      <command_interface name="effort"/>
-      <state_interface name="position"/>
+      <command_interface name="position">
+      </command_interface>
+      <state_interface name="position">
+        <param name="initial_value">1.0</param>
+      </state_interface>
       <state_interface name="velocity"/>
     </joint>
     <joint name="joint_7">
-      <command_interface name="effort"/>
-      <state_interface name="position"/>
+      <command_interface name="position">
+      </command_interface>
+      <state_interface name="position">
+        <param name="initial_value">1.0</param>
+      </state_interface>
       <state_interface name="velocity"/>
     </joint>
   </ros2_control>
-  <!-- Transmission mappings -->
-  <transmission name="tran_1">
-    <type>transmission_interface/SimpleTransmission</type>
-    <joint name="joint_1">
-      <!-- <hardwareInterface>hardware_interface/EffortJointInterface</hardwareInterface> -->
-      <hardwareInterface>effort</hardwareInterface>
-    </joint>
-    <actuator name="motor_1">
-      <!-- <hardwareInterface>hardware_interface/EffortJointInterface</hardwareInterface> -->
-      <hardwareInterface>effort</hardwareInterface>
-      <mechanicalReduction>1</mechanicalReduction>
-    </actuator>
-  </transmission>
-  <transmission name="tran_2">
-    <type>transmission_interface/SimpleTransmission</type>
-    <joint name="joint_2">
-      <!-- <hardwareInterface>hardware_interface/EffortJointInterface</hardwareInterface> -->
-      <hardwareInterface>effort</hardwareInterface>
-    </joint>
-    <actuator name="motor_2">
-      <!-- <hardwareInterface>hardware_interface/EffortJointInterface</hardwareInterface> -->
-      <hardwareInterface>effort</hardwareInterface>
-      <mechanicalReduction>1</mechanicalReduction>
-    </actuator>
-  </transmission>
-  <transmission name="tran_3">
-    <type>transmission_interface/SimpleTransmission</type>
-    <joint name="joint_3">
-      <!-- <hardwareInterface>hardware_interface/EffortJointInterface</hardwareInterface> -->
-      <hardwareInterface>effort</hardwareInterface>
-    </joint>
-    <actuator name="motor_3">
-      <!-- <hardwareInterface>hardware_interface/EffortJointInterface</hardwareInterface> -->
-      <hardwareInterface>effort</hardwareInterface>
-      <mechanicalReduction>1</mechanicalReduction>
-    </actuator>
-  </transmission>
-  <transmission name="tran_4">
-    <type>transmission_interface/SimpleTransmission</type>
-    <joint name="joint_4">
-      <!-- <hardwareInterface>hardware_interface/EffortJointInterface</hardwareInterface> -->
-      <hardwareInterface>effort</hardwareInterface>
-    </joint>
-    <actuator name="motor_4">
-      <!-- <hardwareInterface>hardware_interface/EffortJointInterface</hardwareInterface> -->
-      <hardwareInterface>effort</hardwareInterface>
-      <mechanicalReduction>1</mechanicalReduction>
-    </actuator>
-  </transmission>
-  <transmission name="tran_5">
-    <type>transmission_interface/SimpleTransmission</type>
-    <joint name="joint_5">
-      <!-- <hardwareInterface>hardware_interface/EffortJointInterface</hardwareInterface> -->
-      <hardwareInterface>effort</hardwareInterface>
-    </joint>
-    <actuator name="motor_5">
-      <!-- <hardwareInterface>hardware_interface/EffortJointInterface</hardwareInterface> -->
-      <hardwareInterface>effort</hardwareInterface>
-      <mechanicalReduction>1</mechanicalReduction>
-    </actuator>
-  </transmission>
-  <transmission name="tran_6">
-    <type>transmission_interface/SimpleTransmission</type>
-    <joint name="joint_6">
-      <!-- <hardwareInterface>hardware_interface/EffortJointInterface</hardwareInterface> -->
-      <hardwareInterface>effort</hardwareInterface>
-    </joint>
-    <actuator name="motor_6">
-      <hardwareInterface>effort</hardwareInterface>
-      <mechanicalReduction>1</mechanicalReduction>
-    </actuator>
-  </transmission>
-  <transmission name="tran_7">
-    <type>transmission_interface/SimpleTransmission</type>
-    <joint name="joint_7">
-      <!-- <hardwareInterface>hardware_interface/EffortJointInterface</hardwareInterface> -->
-      <hardwareInterface>effort</hardwareInterface>
-    </joint>
-    <actuator name="motor_7">
-      <!-- <hardwareInterface>hardware_interface/EffortJointInterface</hardwareInterface> -->
-      <hardwareInterface>effort</hardwareInterface>
-      <mechanicalReduction>1</mechanicalReduction>
-    </actuator>
-  </transmission>
   </xacro:macro>
   <xacro:kr810_description />
+  <xacro:arg name="controllers_file" default="BLAH!"/>
   <gazebo>
-    <plugin name="gz_ros2_control" filename="libgz_ros2_control.so"/>
-  </gazebo>
-  <gazebo reference="joint_1">
-    <provideFeedback>true</provideFeedback>
-  </gazebo>
-  <gazebo reference="joint_2">
-    <provideFeedback>true</provideFeedback>
-  </gazebo>
-  <gazebo reference="joint_3">
-    <provideFeedback>true</provideFeedback>
-  </gazebo>
-  <gazebo reference="joint_4">
-    <provideFeedback>true</provideFeedback>
-  </gazebo>
-  <gazebo reference="joint_5">
-    <provideFeedback>true</provideFeedback>
-  </gazebo>
-  <gazebo reference="joint_6">
-    <provideFeedback>true</provideFeedback>
-  </gazebo>
-  <gazebo reference="joint_7">
-    <provideFeedback>true</provideFeedback>
+    <plugin filename="libgz_ros2_control-system.so"
+            name="gz_ros2_control::GazeboSimROS2ControlPlugin">
+      <!-- Point to the controllers YAML we’ll create below -->
+      <!-- <parameters>$(find kr_robot_description)/kr810/config/kr810_controllers.yaml</parameters> -->
+      <parameters>$(arg controllers_file)</parameters>
+      <!-- Optional tuning (documented by gz_ros2_control): -->
+      <!-- <position_proportional_gain>0.3</position_proportional_gain> -->
+      <!-- <hold_joints>true</hold_joints> -->
+    </plugin>
   </gazebo>
 </robot>

Commit message: Resolved a bunch of stuff to work with ros2_control. Still not fully functional

File: kr_robot_description/kr810/urdf/kr810_description.urdf.xacro (robot description, xacro)
@@ -2,4 +2,5 @@
 <robot name="kr2_robot_a810" model="a810" model-revision="051020-0" mechanical-revision="5" features="TIO" xmlns:xacro="http://www.ros.org/wiki/xacro">
   <xacro:macro name="kr810_description">
+  <xacro:property name="kr_robot_description_path" value="package://kr_robot_description/kr810"/>
   <!-- materials -->
   <material name="gray">
@@ -86,5 +87,5 @@
         <origin xyz="0 0 0" rpy="0 0 0" />
         <geometry>
-          <mesh filename="$(find kr_robot_description)/kr810/meshes/a810/a810_Base.stl" scale="0.001 0.001 0.001"/>
+          <mesh filename="${kr_robot_description_path}/meshes/a810/a810_Base.stl" scale="0.001 0.001 0.001"/>
         </geometry>
         <material name="">
@@ -126,5 +127,5 @@
         <origin xyz="0 0 0.169" rpy="0 0 0" />
         <geometry>
-          <mesh filename="$(find kr_robot_description)/kr810/meshes/a810/a810_Link2.stl" scale="0.001 0.001 0.001"/>
+          <mesh filename="${kr_robot_description_path}/meshes/a810/a810_Link2.stl" scale="0.001 0.001 0.001"/>
         </geometry>
         <material name="">
@@ -164,5 +165,5 @@
         <origin xyz="0.049 0 0" rpy="-${pi/2} 0 -${pi/2}" />
         <geometry>
-          <mesh filename="$(find kr_robot_description)/kr810/meshes/a810/a810_Link3.stl" scale="0.001 0.001 0.001"/>
+          <mesh filename="${kr_robot_description_path}/meshes/a810/a810_Link3.stl" scale="0.001 0.001 0.001"/>
         </geometry>
         <material name="">
@@ -188,5 +189,5 @@
         <origin xyz="-0.05 -0.0 0.315" rpy="${pi/2} 0 -${pi/2}" />
         <geometry>
-          <mesh filename="$(find kr_robot_description)/kr810/meshes/a810/a810_Link4.stl" scale="0.001 0.001 0.001"/>
+          <mesh filename="${kr_robot_description_path}/meshes/a810/a810_Link4.stl" scale="0.001 0.001 0.001"/>
         </geometry>
         <material name="">
@@ -226,5 +227,5 @@
         <origin xyz="0.04 0.0005 0.0" rpy="-${pi/2} 0 ${pi/2}" />
         <geometry>
-          <mesh filename="$(find kr_robot_description)/kr810/meshes/a810/a810_Link5.stl" scale="0.001 0.001 0.001"/>
+          <mesh filename="${kr_robot_description_path}/meshes/a810/a810_Link5.stl" scale="0.001 0.001 0.001"/>
         </geometry>
         <material name="">
@@ -247,5 +248,5 @@
         <origin xyz="0.0 0.002 0.1035" rpy="0 0 -${pi/2}" />
         <geometry>
-          <mesh filename="$(find kr_robot_description)/kr810/meshes/a810/a810_Link6.stl" scale="0.001 0.001 0.001"/>
+          <mesh filename="${kr_robot_description_path}/meshes/a810/a810_Link6.stl" scale="0.001 0.001 0.001"/>
         </geometry>
         <material name="">
@@ -287,5 +288,5 @@
         <origin xyz="0.0 0.0 0.0" rpy="0 0 0" />
         <geometry>
-          <mesh filename="$(find kr_robot_description)/kr810/meshes/a810/a810_Link7.stl" scale="0.001 0.001 0.001"/>
+          <mesh filename="${kr_robot_description_path}/meshes/a810/a810_Link7.stl" scale="0.001 0.001 0.001"/>
         </geometry>
         <material name="">
@@ -303,5 +304,5 @@
         <origin xyz="0.0 -0.0 0.0" rpy="0 0 0" />
         <geometry>
-          <mesh filename="$(find kr_robot_description)/kr810/meshes/a810/a810_ToolIO.stl" scale="0.001 0.001 0.001"/>
+          <mesh filename="${kr_robot_description_path}/meshes/a810/a810_ToolIO.stl" scale="0.001 0.001 0.001"/>
         </geometry>
         <material name="">
@@ -429,4 +430,6 @@
     <joint name="joint_1">
       <command_interface name="position">
+        <param name="min">-1</param>
+        <param name="max">1</param>
       </command_interface>
       <state_interface name="position">
@@ -437,4 +440,6 @@
     <joint name="joint_2">
       <command_interface name="position">
+        <param name="min">-1</param>
+        <param name="max">1</param>
       </command_interface>
       <state_interface name="position">
@@ -445,4 +450,6 @@
     <joint name="joint_3">
       <command_interface name="position">
+        <param name="min">-1</param>
+        <param name="max">1</param>
       </command_interface>
       <state_interface name="position">
@@ -453,4 +460,6 @@
     <joint name="joint_4">
       <command_interface name="position">
+        <param name="min">-1</param>
+        <param name="max">1</param>
       </command_interface>
       <state_interface name="position">
@@ -461,4 +470,6 @@
     <joint name="joint_5">
       <command_interface name="position">
+        <param name="min">-1</param>
+        <param name="max">1</param>
       </command_interface>
       <state_interface name="position">
@@ -469,4 +480,6 @@
     <joint name="joint_6">
       <command_interface name="position">
+        <param name="min">-1</param>
+        <param name="max">1</param>
       </command_interface>
       <state_interface name="position">
@@ -477,4 +490,6 @@
     <joint name="joint_7">
       <command_interface name="position">
+        <param name="min">-1</param>
+        <param name="max">1</param>
       </command_interface>
       <state_interface name="position">
@@ -491,5 +506,4 @@
             name="gz_ros2_control::GazeboSimROS2ControlPlugin">
       <!-- Point to the controllers YAML we’ll create below -->
-      <!-- <parameters>$(find kr_robot_description)/kr810/config/kr810_controllers.yaml</parameters> -->
       <parameters>$(arg controllers_file)</parameters>
       <!-- Optional tuning (documented by gz_ros2_control): -->
